Commit message: Added model with inertias. Can visualize in RViz

File: description/urdf/cybertruck.urdf.xacro (robot description, xacro)
@@ -1,11 +1,15 @@
 <?xml version="1.0"?>
 <robot name="cybertruck" xmlns:xacro="http://ros.org/wiki/xacro">
+    <!-- Includes -->
+    <xacro:include filename="$(find description)/urdf/constants.xacro"/>
+    <xacro:include filename="$(find description)/urdf/inertias.xacro"/>
     <link name="base_link"/>
     <!-- Body -->
+    <!-- NOTE: cybertuck uses a frame where "-y" is forward for the model. base_link -> body_link will correct for this -->
     <link name="body_link">
         <visual>
             <origin xyz="0 0 0" rpy="0 0 0"/>
             <geometry>
-                <mesh filename="package://description/urdf/meshes/cybertruck_body.stl"/>
+                <mesh filename="package://description/urdf/meshes/cybertruck_body.dae"/>
             </geometry>
         </visual>
@@ -13,12 +17,117 @@
             <origin xyz="0 0 0" rpy="0 0 0"/>
             <geometry>
-                <mesh filename="package://description/urdf/meshes/cybertruck_body.stl"/>
+                <mesh filename="package://description/urdf/meshes/cybertruck_body.dae"/>
             </geometry>
         </collision>
+        <inertial>
+            <mass value="${body_mass}"/>
+            <xacro:body_inertia mass="${body_mass}" length="${body_length}" width="${body_width}" height="${body_height}"/>
+        </inertial>
     </link>
     <joint name="body_joint" type="fixed">
         <parent link="base_link"/>
         <child link="body_link"/>
-        <origin xyz="0 0 0.2" rpy="0 0 0"/>
+        <origin xyz="0 0 0.0" rpy="0 0 ${pi / 2}"/>
+    </joint>
+    <!-- Wheels -->
+    <!-- Front Left Wheel -->
+    <link name="front_left_wheel_link">
+        <visual>
+            <origin xyz="0 0 0" rpy="0 0 0"/>
+            <geometry>
+                <mesh filename="package://description/urdf/meshes/cybertruck_left_wheel.dae"/>
+            </geometry>
+        </visual>
+        <collision>
+            <origin xyz="0 0 0" rpy="0 0 0"/>
+            <geometry>
+                <mesh filename="package://description/urdf/meshes/cybertruck_left_wheel.dae"/>
+            </geometry>
+        </collision>
+        <inertial>
+            <mass value="${wheel_mass}"/>
+            <xacro:wheel_inertia mass="${wheel_mass}" length="${wheel_width}" radius="${wheel_radius}"/>
+        </inertial>
+    </link>
+    <joint name="front_left_wheel_joint" type="continuous">
+        <parent link="body_link"/>
+        <child link="front_left_wheel_link"/>
+        <origin xyz="${left_wheel} ${front_wheel} ${height_to_wheel}" rpy="0 0 0"/>
+        <axis xyz="1 0 0"/>
+    </joint>
+    <!-- Back Left Wheel -->
+    <link name="back_left_wheel_link">
+        <visual>
+            <origin xyz="0 0 0" rpy="0 0 0"/>
+            <geometry>
+                <mesh filename="package://description/urdf/meshes/cybertruck_left_wheel.dae"/>
+            </geometry>
+        </visual>
+        <collision>
+            <origin xyz="0 0 0" rpy="0 0 0"/>
+            <geometry>
+                <mesh filename="package://description/urdf/meshes/cybertruck_left_wheel.dae"/>
+            </geometry>
+        </collision>
+        <inertial>
+            <mass value="${wheel_mass}"/>
+            <xacro:wheel_inertia mass="${wheel_mass}" length="${wheel_width}" radius="${wheel_radius}"/>
+        </inertial>
+    </link>
+    <joint name="back_left_wheel_joint" type="continuous">
+        <parent link="body_link"/>
+        <child link="back_left_wheel_link"/>
+        <origin xyz="${left_wheel} ${back_wheel} ${height_to_wheel}" rpy="0 0 0"/>
+        <axis xyz="1 0 0"/>
+    </joint>
+    <!-- Front Right Wheel -->
+    <link name="front_right_wheel_link">
+        <visual>
+            <origin xyz="0 0 0" rpy="0 0 0"/>
+            <geometry>
+                <mesh filename="package://description/urdf/meshes/cybertruck_right_wheel.dae"/>
+            </geometry>
+        </visual>
+        <collision>
+            <origin xyz="0 0 0" rpy="0 0 0"/>
+            <geometry>
+                <mesh filename="package://description/urdf/meshes/cybertruck_right_wheel.dae"/>
+            </geometry>
+        </collision>
+        <inertial>
+            <mass value="${wheel_mass}"/>
+            <xacro:wheel_inertia mass="${wheel_mass}" length="${wheel_width}" radius="${wheel_radius}"/>
+        </inertial>
+    </link>
+    <joint name="front_right_wheel_joint" type="continuous">
+        <parent link="body_link"/>
+        <child link="front_right_wheel_link"/>
+        <origin xyz="${right_wheel} ${front_wheel} ${height_to_wheel}" rpy="0 0 0"/>
+        <axis xyz="1 0 0"/>
+    </joint>
+    <!-- Back Right Wheel -->
+    <link name="back_right_wheel_link">
+        <visual>
+            <origin xyz="0 0 0" rpy="0 0 0"/>
+            <geometry>
+                <mesh filename="package://description/urdf/meshes/cybertruck_right_wheel.dae"/>
+            </geometry>
+        </visual>
+        <collision>
+            <origin xyz="0 0 0" rpy="0 0 0"/>
+            <geometry>
+                <mesh filename="package://description/urdf/meshes/cybertruck_right_wheel.dae"/>
+            </geometry>
+        </collision>
+        <inertial>
+            <mass value="${wheel_mass}"/>
+            <xacro:wheel_inertia mass="${wheel_mass}" length="${wheel_width}" radius="${wheel_radius}"/>
+        </inertial>
+    </link>
+    <joint name="back_right_wheel_joint" type="continuous">
+        <parent link="body_link"/>
+        <child link="back_right_wheel_link"/>
+        <origin xyz="${right_wheel} ${back_wheel} ${height_to_wheel}" rpy="0 0 0"/>
+        <axis xyz="1 0 0"/>
     </joint>
 </robot>

Commit message: Macro for wheels and planar movement controller

File: description/urdf/cybertruck.urdf.xacro (robot description, xacro)
@@ -21,8 +21,4 @@
             </geometry>
         </collision>
-        <inertial>
-            <mass value="${body_mass}"/>
-            <xacro:body_inertia mass="${body_mass}" length="${body_length}" width="${body_width}" height="${body_height}"/>
-        </inertial>
     </link>
     <joint name="body_joint" type="fixed">
@@ -32,117 +28,4 @@
     </joint>
     <!-- Wheels -->
-    <!-- Motor Transmissions -->
-    <xacro:macro name="Transmission" params="joint">
-        <transmission name="trans_${joint}">
-            <type>transmission_interface/SimpleTransmission</type>
-            <joint name="${joint}">
-                <hardwareInterface>hardware_interface/EffortJointInterface</hardwareInterface>
-            </joint>
-            <actuator name="${joint}_motor"/>
-        </transmission>
-    </xacro:macro>
-    <!-- Front Left Wheel -->
-    <link name="front_left_wheel_link">
-        <visual>
-            <origin xyz="0 0 0" rpy="0 0 0"/>
-            <geometry>
-                <mesh filename="package://description/urdf/meshes/cybertruck_left_wheel.dae"/>
-            </geometry>
-        </visual>
-        <collision>
-            <origin xyz="0 0 0" rpy="0 ${pi / 2.0} 0"/>
-            <geometry>
-                <cylinder length="${wheel_width}" radius="${wheel_radius}"/>
-            </geometry>
-        </collision>
-        <inertial>
-            <mass value="${wheel_mass}"/>
-            <xacro:wheel_inertia mass="${wheel_mass}" length="${wheel_width}" radius="${wheel_radius}"/>
-        </inertial>
-    </link>
-    <joint name="front_left_wheel_joint" type="continuous">
-        <parent link="body_link"/>
-        <child link="front_left_wheel_link"/>
-        <origin xyz="${left_wheel} ${front_wheel} ${height_to_wheel}" rpy="0 0 0"/>
-        <axis xyz="1 0 0"/>
-    </joint>
-    <xacro:Transmission joint="front_left_wheel_joint"/>
-    <!-- Back Left Wheel -->
-    <link name="back_left_wheel_link">
-        <visual>
-            <origin xyz="0 0 0" rpy="0 0 0"/>
-            <geometry>
-                <mesh filename="package://description/urdf/meshes/cybertruck_left_wheel.dae"/>
-            </geometry>
-        </visual>
-        <collision>
-            <origin xyz="0 0 0" rpy="0 ${pi / 2.0} 0"/>
-            <geometry>
-                <cylinder length="${wheel_width}" radius="${wheel_radius}"/>
-            </geometry>
-        </collision>
-        <inertial>
-            <mass value="${wheel_mass}"/>
-            <xacro:wheel_inertia mass="${wheel_mass}" length="${wheel_width}" radius="${wheel_radius}"/>
-        </inertial>
-    </link>
-    <joint name="back_left_wheel_joint" type="continuous">
-        <parent link="body_link"/>
-        <child link="back_left_wheel_link"/>
-        <origin xyz="${left_wheel} ${back_wheel} ${height_to_wheel}" rpy="0 0 0"/>
-        <axis xyz="1 0 0"/>
-    </joint>
-    <!-- <xacro:Transmission joint="back_left_wheel_joint"/> -->
-    <!-- Front Right Wheel -->
-    <link name="front_right_wheel_link">
-        <visual>
-            <origin xyz="0 0 0" rpy="0 0 0"/>
-            <geometry>
-                <mesh filename="package://description/urdf/meshes/cybertruck_right_wheel.dae"/>
-            </geometry>
-        </visual>
-        <collision>
-            <origin xyz="0 0 0" rpy="0 ${pi / 2.0} 0"/>
-            <geometry>
-                <cylinder length="${wheel_width}" radius="${wheel_radius}"/>
-            </geometry>
-        </collision>
-        <inertial>
-            <mass value="${wheel_mass}"/>
-            <xacro:wheel_inertia mass="${wheel_mass}" length="${wheel_width}" radius="${wheel_radius}"/>
-        </inertial>
-    </link>
-    <joint name="front_right_wheel_joint" type="continuous">
-        <parent link="body_link"/>
-        <child link="front_right_wheel_link"/>
-        <origin xyz="${right_wheel} ${front_wheel} ${height_to_wheel}" rpy="0 0 0"/>
-        <axis xyz="1 0 0"/>
-    </joint>
-    <xacro:Transmission joint="front_right_wheel_joint"/>
-    <!-- Back Right Wheel -->
-    <link name="back_right_wheel_link">
-        <visual>
-            <origin xyz="0 0 0" rpy="0 0 0"/>
-            <geometry>
-                <mesh filename="package://description/urdf/meshes/cybertruck_right_wheel.dae"/>
-            </geometry>
-        </visual>
-        <collision>
-            <origin xyz="0 0 0" rpy="0 ${pi / 2.0} 0"/>
-            <geometry>
-                <cylinder length="${wheel_width}" radius="${wheel_radius}"/>
-            </geometry>
-        </collision>
-        <inertial>
-            <mass value="${wheel_mass}"/>
-            <xacro:wheel_inertia mass="${wheel_mass}" length="${wheel_width}" radius="${wheel_radius}"/>
-        </inertial>
-    </link>
-    <joint name="back_right_wheel_joint" type="continuous">
-        <parent link="body_link"/>
-        <child link="back_right_wheel_link"/>
-        <origin xyz="${right_wheel} ${back_wheel} ${height_to_wheel}" rpy="0 0 0"/>
-        <axis xyz="1 0 0"/>
-    </joint>
-    <!-- <xacro:Transmission joint="back_right_wheel_joint"/> -->
+    <xacro:include filename="$(find description)/urdf/wheels.urdf.xacro"/>
 </robot>

File: description/urdf/inertias.xacro (robot description, xacro)
@@ -19,3 +19,11 @@
         />
     </xacro:macro>
+    <!-- Sphere -->
+    <xacro:macro name="sphere_inertia" params="mass radius">
+        <inertia
+            ixx="${(2.0 * mass * radius * radius) / 5.0}" ixy="0.0" ixz="0.0"
+            iyx="0.0" iyy="${(2.0 * mass * radius * radius) / 5.0}" iyz="0.0"
+            izx="0.0" izy="0.0" izz="${(2.0 * mass * radius * radius) / 5.0}"
+        />
+    </xacro:macro>
 </robot>

File: description/urdf/plugins.gazebo.xacro (robot description, xacro)
@@ -4,38 +4,63 @@
     <xacro:include filename="$(find description)/urdf/constants.xacro"/>
     <!-- Differential Drive Controller -->
-    <gazebo>
+    <!-- <gazebo>
         <plugin name="differential_drive_controller" filename="libgazebo_ros_diff_drive.so">
             <alwaysOn>true</alwaysOn>
             <legacyMode>false</legacyMode>
-            <rosDebugLevel>na</rosDebugLevel>
+            <rosDebugLevel>na</rosDebugLevel> -->
             <!-- Plugin update rate (Hz) -->
-            <updateRate>30</updateRate>
+            <!-- <updateRate>30</updateRate> -->
             <!-- Name of joints connecting to wheels -->
-            <leftJoint>front_left_wheel_joint</leftJoint>
-            <rightJoint>front_right_wheel_joint</rightJoint>
+            <!-- <leftJoint>front_left_wheel_joint</leftJoint>
+            <rightJoint>front_right_wheel_joint</rightJoint> -->
             <!-- Wheel properties -->
-            <wheelSeparation>${wheel_separation}</wheelSeparation>
+            <!-- <wheelSeparation>${wheel_separation}</wheelSeparation>
             <wheelDiameter>${2.0 * wheel_radius}</wheelDiameter>
             <wheelAcceleration>0</wheelAcceleration>
             <wheelTorque>5</wheelTorque>
-            <torque>5</torque>
+            <torque>5</torque> -->
             <!-- Topic to receive geometry_msgs/Twist message commands -->
-            <commandTopic>cmd_vel</commandTopic>
+            <!-- <commandTopic>cmd_vel</commandTopic> -->
             <!-- Odometry (nav_msgs/Odometry) settings -->
-            <odometrySource>world</odometrySource>
+            <!-- <odometrySource>world</odometrySource>
             <odometryTopic>odom</odometryTopic>
-            <odometryFrame>odom</odometryFrame>
+            <odometryFrame>odom</odometryFrame> -->
             <!-- Robot frame to calculate odometry from -->
-            <robotBaseFrame>base_link</robotBaseFrame>
+            <!-- <robotBaseFrame>base_link</robotBaseFrame> -->
             <!-- Publish TF frames -->
-            <publishTf>true</publishTf>
+            <!-- <publishTf>true</publishTf>
             <publishOdomTF>true</publishOdomTF>
             <publishWheelTF>false</publishWheelTF>
             <publishWheelJointState>true</publishWheelJointState>
         </plugin>
+    </gazebo> -->
+    <!-- <gazebo>
+        <plugin name="skid_steer_drive_controller" filename="libgazebo_ros_skid_steer_drive.so">
+            <updateRate>30.0</updateRate>
+            <robotNamespace>/</robotNamespace>
+            <leftFrontJoint>front_left_wheel_joint</leftFrontJoint>
+            <rightFrontJoint>front_right_wheel_joint</rightFrontJoint>
+            <leftRearJoint>back_left_wheel_joint</leftRearJoint>
+            <rightRearJoint>back_right_wheel_joint</rightRearJoint>
+            <wheelSeparation>${wheel_separation}</wheelSeparation>
+            <wheelDiameter>${2.0 * wheel_radius}</wheelDiameter>
+            <robotBaseFrame>base_link</robotBaseFrame>
+            <torque>20</torque>
+            <topicName>cmd_vel</topicName>
+            <broadcastTF>false</broadcastTF>
+        </plugin>
+    </gazebo> -->
+    <gazebo>
+        <plugin name="object_controller" filename="libgazebo_ros_planar_move.so">
+            <commandTopic>cmd_vel</commandTopic>
+            <odometryTopic>odom</odometryTopic>
+            <odometryFrame>odom</odometryFrame>
+            <odometryRate>20.0</odometryRate>
+            <robotBaseFrame>base_link</robotBaseFrame>
+        </plugin>
     </gazebo>
     <!-- lets all the transmission tags be read -->
-    <gazebo>
+    <!-- <gazebo>
         <plugin name="gazebo_ros_control" filename="libgazebo_ros_control.so"/>
-    </gazebo>
+    </gazebo> -->
 </robot>

Commit message: Added back inertial tag for body_link

File: description/urdf/cybertruck.urdf.xacro (robot description, xacro)
@@ -21,4 +21,8 @@
             </geometry>
         </collision>
+        <inertial>
+            <mass value="${body_mass}"/>
+            <xacro:body_inertia mass="${body_mass}" length="${body_length}" width="${body_width}" height="${body_height}"/>
+        </inertial>
     </link>
     <joint name="body_joint" type="fixed">
