Commit message: Added range sensor plugin and cleaned up code

File: description/urdf/cybertruck.urdf.xacro (robot description, xacro)
@@ -33,3 +33,10 @@
     <!-- Wheels -->
     <xacro:include filename="$(find description)/urdf/wheels.urdf.xacro"/>
+    <!-- IR Sensor -->
+    <link name="base_ir_link"/>
+    <joint name="base_ir_joint" type="fixed">
+        <parent link="body_link"/>
+        <child link="base_ir_link"/>
+        <origin xyz="0 ${front_wheel} ${-height_to_wheel}" rpy="0 0 ${-pi / 2}"/>
+    </joint>
 </robot>

File: description/urdf/plugins.gazebo.xacro (robot description, xacro)
@@ -3,52 +3,5 @@
     <!-- Constants -->
     <xacro:include filename="$(find description)/urdf/constants.xacro"/>
-    <!-- Differential Drive Controller -->
-    <!-- <gazebo>
-        <plugin name="differential_drive_controller" filename="libgazebo_ros_diff_drive.so">
-            <alwaysOn>true</alwaysOn>
-            <legacyMode>false</legacyMode>
-            <rosDebugLevel>na</rosDebugLevel> -->
-            <!-- Plugin update rate (Hz) -->
-            <!-- <updateRate>30</updateRate> -->
-            <!-- Name of joints connecting to wheels -->
-            <!-- <leftJoint>front_left_wheel_joint</leftJoint>
-            <rightJoint>front_right_wheel_joint</rightJoint> -->
-            <!-- Wheel properties -->
-            <!-- <wheelSeparation>${wheel_separation}</wheelSeparation>
-            <wheelDiameter>${2.0 * wheel_radius}</wheelDiameter>
-            <wheelAcceleration>0</wheelAcceleration>
-            <wheelTorque>5</wheelTorque>
-            <torque>5</torque> -->
-            <!-- Topic to receive geometry_msgs/Twist message commands -->
-            <!-- <commandTopic>cmd_vel</commandTopic> -->
-            <!-- Odometry (nav_msgs/Odometry) settings -->
-            <!-- <odometrySource>world</odometrySource>
-            <odometryTopic>odom</odometryTopic>
-            <odometryFrame>odom</odometryFrame> -->
-            <!-- Robot frame to calculate odometry from -->
-            <!-- <robotBaseFrame>base_link</robotBaseFrame> -->
-            <!-- Publish TF frames -->
-            <!-- <publishTf>true</publishTf>
-            <publishOdomTF>true</publishOdomTF>
-            <publishWheelTF>false</publishWheelTF>
-            <publishWheelJointState>true</publishWheelJointState>
-        </plugin>
-    </gazebo> -->
-    <!-- <gazebo>
-        <plugin name="skid_steer_drive_controller" filename="libgazebo_ros_skid_steer_drive.so">
-            <updateRate>30.0</updateRate>
-            <robotNamespace>/</robotNamespace>
-            <leftFrontJoint>front_left_wheel_joint</leftFrontJoint>
-            <rightFrontJoint>front_right_wheel_joint</rightFrontJoint>
-            <leftRearJoint>back_left_wheel_joint</leftRearJoint>
-            <rightRearJoint>back_right_wheel_joint</rightRearJoint>
-            <wheelSeparation>${wheel_separation}</wheelSeparation>
-            <wheelDiameter>${2.0 * wheel_radius}</wheelDiameter>
-            <robotBaseFrame>base_link</robotBaseFrame>
-            <torque>20</torque>
-            <topicName>cmd_vel</topicName>
-            <broadcastTF>false</broadcastTF>
-        </plugin>
-    </gazebo> -->
+    <!-- Planar Move Controller -->
     <gazebo>
         <plugin name="object_controller" filename="libgazebo_ros_planar_move.so">
@@ -56,11 +9,49 @@
             <odometryTopic>odom</odometryTopic>
             <odometryFrame>odom</odometryFrame>
-            <odometryRate>20.0</odometryRate>
+            <odometryRate>30.0</odometryRate>
             <robotBaseFrame>base_link</robotBaseFrame>
         </plugin>
     </gazebo>
-    <!-- lets all the transmission tags be read -->
-    <!-- <gazebo>
+    <!-- ROS Control: Reads transmission tags -->
+    <gazebo>
         <plugin name="gazebo_ros_control" filename="libgazebo_ros_control.so"/>
-    </gazebo> -->
+    </gazebo>
+    <!-- IR Sensor: Range Sensor -->
+    <gazebo reference="base_ir_link">
+        <sensor type="ray" name="RangeSensor">
+            <pose>0 0 0 0 0 0</pose>
+            <visualize>false</visualize>
+            <update_rate>50</update_rate>
+            <ray>
+                <scan>
+                <horizontal>
+                    <samples>10</samples>
+                    <resolution>1</resolution>
+                    <min_angle>-0.14835</min_angle>
+                    <max_angle>0.14835</max_angle>
+                </horizontal>
+                <vertical>
+                    <samples>10</samples>
+                    <resolution>1</resolution>
+                    <min_angle>-0.14835</min_angle>
+                    <max_angle>0.14835</max_angle>
+                </vertical>
+                </scan>
+                <range>
+                <min>0.01</min>
+                <max>2</max>
+                <resolution>0.02</resolution>
+                </range>
+            </ray>
+            <plugin filename="libgazebo_ros_range.so" name="gazebo_ros_range">
+                <gaussianNoise>0.005</gaussianNoise>
+                <alwaysOn>true</alwaysOn>
+                <updateRate>50</updateRate>
+                <topicName>sensor/ir</topicName>
+                <frameName>base_ir_link</frameName>
+                <radiation>INFRARED</radiation>
+                <fov>0.2967</fov>
+            </plugin>
+        </sensor>
+    </gazebo>
 </robot>

File: description/urdf/wheels.urdf.xacro (robot description, xacro)
@@ -4,4 +4,14 @@
     <xacro:include filename="$(find description)/urdf/constants.xacro"/>
     <xacro:include filename="$(find description)/urdf/inertias.xacro"/>
+    <!-- Motor Transmissions -->
+    <xacro:macro name="Transmission" params="joint">
+        <transmission name="trans_${joint}">
+            <type>transmission_interface/SimpleTransmission</type>
+            <joint name="${joint}">
+                <hardwareInterface>hardware_interface/EffortJointInterface</hardwareInterface>
+            </joint>
+            <actuator name="${joint}_motor"/>
+        </transmission>
+    </xacro:macro>
     <!-- Wheel macro -->
     <xacro:macro name="Wheel" params="fb lr">
@@ -10,6 +20,4 @@
                 <origin xyz="0 0 0" rpy="0 0 0"/>
                 <geometry>
-                    <!-- <sphere radius="${wheel_radius}"/> -->
-                    <!-- <cylinder length="${wheel_width}" radius="${wheel_radius}"/> -->
                     <mesh filename="package://description/urdf/meshes/cybertruck_${lr}_wheel.dae"/>
                 </geometry>
@@ -18,6 +26,4 @@
                 <origin xyz="0 0 0" rpy="0 ${pi/2} 0"/>
                 <geometry>
-                    <!-- <box size="${wheel_radius} ${wheel_radius} ${wheel_radius}"/> -->
-                    <!-- <sphere radius="${wheel_radius}"/> -->
                     <cylinder length="${wheel_width}" radius="${wheel_radius}"/>
                 </geometry>
@@ -25,6 +31,4 @@
             <inertial>
                 <mass value="${wheel_mass}"/>
-                <!-- <xacro:body_inertia mass="${wheel_mass}" length="${wheel_radius}" width="${wheel_radius}" height="${wheel_radius}"/> -->
-                <!-- <xacro:sphere_inertia mass="${wheel_mass}" radius="${wheel_radius}"/> -->
                 <xacro:wheel_inertia mass="${wheel_mass}" length="${wheel_width}" radius="${wheel_radius}"/>
             </inertial>
@@ -36,4 +40,5 @@
             <axis xyz="1 0 0"/>
         </joint>
+        <xacro:Transmission joint="${fb}_${lr}_wheel_joint"/>
     </xacro:macro>
     <!-- Instantiate wheels -->

Commit message: Added light (illuminance) sensor package/plugin

File: description/urdf/cybertruck.urdf.xacro (robot description, xacro)
@@ -40,3 +40,16 @@
         <origin xyz="0 ${front_wheel} ${-height_to_wheel}" rpy="0 0 ${-pi / 2}"/>
     </joint>
+    <!-- Illuminance Sensor -->
+    <link name="light_link"/>
+    <joint name="light_joint" type="fixed">
+        <parent link="body_link"/>
+        <child link="light_link"/>
+        <origin xyz="0 ${-body_length} 0" rpy="0 ${pi / 2} ${pi / 2}"/>
+    </joint>
+    <link name="light_link_optical"/>
+    <joint name="light_optical_joint" type="fixed">
+        <parent link="light_link"/>
+        <child link="light_link_optical"/>
+        <origin xyz="0 0 0" rpy="${-pi/2} 0 ${-pi/2}"/>
+    </joint>
 </robot>

File: description/urdf/plugins.gazebo.xacro (robot description, xacro)
@@ -78,3 +78,37 @@
         </sensor>
     </gazebo>
+    <!-- Illuminance Sensor: Inherits from Camera -->
+    <!-- NOTE: illuminance only published if the image topic is being read from! -->
+    <gazebo reference="light_link">
+        <sensor name='light_sensor' type='camera'>
+            <camera name='light_sensor'>
+                <horizontal_fov>1.047</horizontal_fov>
+                <image>
+                    <width>320</width>
+                    <height>240</height>
+                    <format>R8G8B8</format>
+                </image>
+                <clip>
+                    <near>0.01</near>
+                    <far>10</far>
+                </clip>
+            </camera>
+            <plugin name="gazebo_light_sensor_plugin" filename="libgazebo_light_sensor_plugin.so">
+                <cameraName>light_sensor</cameraName>
+                <alwaysOn>true</alwaysOn>
+                <updateRate>10</updateRate>
+                <imageTopicName>rgb/image_raw</imageTopicName>
+                <depthImageTopicName>depth/image_raw</depthImageTopicName>
+                <pointCloudTopicName>depth/points</pointCloudTopicName>
+                <cameraInfoTopicName>rgb/camera_info</cameraInfoTopicName>
+                <depthImageCameraInfoTopicName>depth/camera_info</depthImageCameraInfoTopicName>
+                <frameName>light_link_optical</frameName>
+                <distortion_K1>0.0</distortion_K1>
+                <distortion_K2>0.0</distortion_K2>
+                <distortion_K3>0.0</distortion_K3>
+                <distortion_T1>0.0</distortion_T1>
+                <distortion_T2>0.0</distortion_T2>
+            </plugin>
+        </sensor>
+    </gazebo>
 </robot>
