Commit message: Added diff drive motor controller plugin. Can issue cmd_vel and publish odom frame

File: description/urdf/constants.xacro (robot description, xacro)
@@ -16,3 +16,4 @@
     <xacro:property name="wheel_radius" value="0.01"/>
     <xacro:property name="wheel_width" value="0.006"/>
+    <xacro:property name="wheel_separation" value="0.047"/>
 </robot>

File: description/urdf/cybertruck.urdf.xacro (robot description, xacro)
@@ -4,4 +4,5 @@
     <xacro:include filename="$(find description)/urdf/constants.xacro"/>
     <xacro:include filename="$(find description)/urdf/inertias.xacro"/>
+    <xacro:include filename="$(find description)/urdf/plugins.gazebo.xacro"/>
     <link name="base_link"/>
     <!-- Body -->
@@ -31,4 +32,14 @@
     </joint>
     <!-- Wheels -->
+    <!-- Motor Transmissions -->
+    <xacro:macro name="Transmission" params="joint">
+        <transmission name="trans_${joint}">
+            <type>transmission_interface/SimpleTransmission</type>
+            <joint name="${joint}">
+                <hardwareInterface>hardware_interface/EffortJointInterface</hardwareInterface>
+            </joint>
+            <actuator name="${joint}_motor"/>
+        </transmission>
+    </xacro:macro>
     <!-- Front Left Wheel -->
     <link name="front_left_wheel_link">
@@ -40,7 +51,7 @@
         </visual>
         <collision>
-            <origin xyz="0 0 0" rpy="0 0 0"/>
+            <origin xyz="0 0 0" rpy="0 ${pi / 2.0} 0"/>
             <geometry>
-                <mesh filename="package://description/urdf/meshes/cybertruck_left_wheel.dae"/>
+                <cylinder length="${wheel_width}" radius="${wheel_radius}"/>
             </geometry>
         </collision>
@@ -56,4 +67,5 @@
         <axis xyz="1 0 0"/>
     </joint>
+    <xacro:Transmission joint="front_left_wheel_joint"/>
     <!-- Back Left Wheel -->
     <link name="back_left_wheel_link">
@@ -65,7 +77,7 @@
         </visual>
         <collision>
-            <origin xyz="0 0 0" rpy="0 0 0"/>
+            <origin xyz="0 0 0" rpy="0 ${pi / 2.0} 0"/>
             <geometry>
-                <mesh filename="package://description/urdf/meshes/cybertruck_left_wheel.dae"/>
+                <cylinder length="${wheel_width}" radius="${wheel_radius}"/>
             </geometry>
         </collision>
@@ -81,4 +93,5 @@
         <axis xyz="1 0 0"/>
     </joint>
+    <xacro:Transmission joint="back_left_wheel_joint"/>
     <!-- Front Right Wheel -->
     <link name="front_right_wheel_link">
@@ -90,7 +103,7 @@
         </visual>
         <collision>
-            <origin xyz="0 0 0" rpy="0 0 0"/>
+            <origin xyz="0 0 0" rpy="0 ${pi / 2.0} 0"/>
             <geometry>
-                <mesh filename="package://description/urdf/meshes/cybertruck_right_wheel.dae"/>
+                <cylinder length="${wheel_width}" radius="${wheel_radius}"/>
             </geometry>
         </collision>
@@ -106,4 +119,5 @@
         <axis xyz="1 0 0"/>
     </joint>
+    <xacro:Transmission joint="front_right_wheel_joint"/>
     <!-- Back Right Wheel -->
     <link name="back_right_wheel_link">
@@ -115,7 +129,7 @@
         </visual>
         <collision>
-            <origin xyz="0 0 0" rpy="0 0 0"/>
+            <origin xyz="0 0 0" rpy="0 ${pi / 2.0} 0"/>
             <geometry>
-                <mesh filename="package://description/urdf/meshes/cybertruck_right_wheel.dae"/>
+                <cylinder length="${wheel_width}" radius="${wheel_radius}"/>
             </geometry>
         </collision>
@@ -131,3 +145,4 @@
         <axis xyz="1 0 0"/>
     </joint>
+    <xacro:Transmission joint="back_right_wheel_joint"/>
 </robot>

Commit message: Robot moves well forward/backwards. Doesn't work when trying to turn

File: description/urdf/constants.xacro (robot description, xacro)
@@ -8,10 +8,10 @@
     <xacro:property name="height_to_wheel" value="-0.015"/>
     <!-- Body properties -->
-    <xacro:property name="body_mass" value="3.0"/>
+    <xacro:property name="body_mass" value="2.5"/>
     <xacro:property name="body_length" value="0.14"/>
     <xacro:property name="body_width" value="0.05"/>
     <xacro:property name="body_height" value="0.04"/>
     <!-- Wheels properties -->
-    <xacro:property name="wheel_mass" value="0.125"/>
+    <xacro:property name="wheel_mass" value="0.05"/>
     <xacro:property name="wheel_radius" value="0.01"/>
     <xacro:property name="wheel_width" value="0.006"/>

File: description/urdf/cybertruck.urdf.xacro (robot description, xacro)
@@ -93,5 +93,5 @@
         <axis xyz="1 0 0"/>
     </joint>
-    <xacro:Transmission joint="back_left_wheel_joint"/>
+    <!-- <xacro:Transmission joint="back_left_wheel_joint"/> -->
     <!-- Front Right Wheel -->
     <link name="front_right_wheel_link">
@@ -145,4 +145,4 @@
         <axis xyz="1 0 0"/>
     </joint>
-    <xacro:Transmission joint="back_right_wheel_joint"/>
+    <!-- <xacro:Transmission joint="back_right_wheel_joint"/> -->
 </robot>

File: description/urdf/plugins.gazebo.xacro (robot description, xacro)
@@ -3,12 +3,16 @@
     <!-- Constants -->
     <xacro:include filename="$(find description)/urdf/constants.xacro"/>
-    <!-- Differential Drive -->
+    <!-- Differential Drive Controller -->
     <gazebo>
         <plugin name="differential_drive_controller" filename="libgazebo_ros_diff_drive.so">
             <alwaysOn>true</alwaysOn>
+            <legacyMode>false</legacyMode>
+            <rosDebugLevel>na</rosDebugLevel>
+            <!-- Plugin update rate (Hz) -->
             <updateRate>30</updateRate>
-            <legacyMode>false</legacyMode>
+            <!-- Name of joints connecting to wheels -->
             <leftJoint>front_left_wheel_joint</leftJoint>
             <rightJoint>front_right_wheel_joint</rightJoint>
+            <!-- Wheel properties -->
             <wheelSeparation>${wheel_separation}</wheelSeparation>
             <wheelDiameter>${2.0 * wheel_radius}</wheelDiameter>
@@ -16,14 +20,17 @@
             <wheelTorque>5</wheelTorque>
             <torque>5</torque>
+            <!-- Topic to receive geometry_msgs/Twist message commands -->
             <commandTopic>cmd_vel</commandTopic>
+            <!-- Odometry (nav_msgs/Odometry) settings -->
             <odometrySource>world</odometrySource>
             <odometryTopic>odom</odometryTopic>
             <odometryFrame>odom</odometryFrame>
+            <!-- Robot frame to calculate odometry from -->
             <robotBaseFrame>base_link</robotBaseFrame>
+            <!-- Publish TF frames -->
             <publishTf>true</publishTf>
             <publishOdomTF>true</publishOdomTF>
             <publishWheelTF>false</publishWheelTF>
             <publishWheelJointState>true</publishWheelJointState>
-            <rosDebugLevel>na</rosDebugLevel>
         </plugin>
     </gazebo>

Commit message: Fixed turning issue by removing friction from rear wheels. Cleaned up some files

File: description/urdf/constants.xacro (robot description, xacro)
@@ -1,10 +1,4 @@
 <?xml version="1.0"?>
 <robot name="constants" xmlns:xacro="http://ros.org/wiki/xacro">
-    <!-- Distances from Body to Wheels -->
-    <xacro:property name="front_wheel" value="-0.053"/>
-    <xacro:property name="back_wheel" value="0.04"/>
-    <xacro:property name="right_wheel" value="-0.0235"/>
-    <xacro:property name="left_wheel" value="0.0235"/>
-    <xacro:property name="height_to_wheel" value="-0.015"/>
     <!-- Body properties -->
     <xacro:property name="body_mass" value="2.5"/>
@@ -17,3 +11,9 @@
     <xacro:property name="wheel_width" value="0.006"/>
     <xacro:property name="wheel_separation" value="0.047"/>
+    <!-- Distances from Body to Wheels -->
+    <xacro:property name="front_wheel" value="-0.053"/>
+    <xacro:property name="back_wheel" value="0.04"/>
+    <xacro:property name="right_wheel" value="-${wheel_separation/2}"/>
+    <xacro:property name="left_wheel" value="${wheel_separation/2}"/>
+    <xacro:property name="height_to_wheel" value="-0.015"/>
 </robot>

File: description/urdf/cybertruck.urdf.xacro (robot description, xacro)
@@ -22,6 +22,5 @@
         </collision>
         <inertial>
-            <mass value="${body_mass}"/>
-            <xacro:body_inertia mass="${body_mass}" length="${body_length}" width="${body_width}" height="${body_height}"/>
+            <xacro:body_inertial m="${body_mass}" l="${body_length}" w="${body_width}" h="${body_height}"/>
         </inertial>
     </link>

File: description/urdf/inertias.xacro (robot description, xacro)
@@ -3,26 +3,20 @@
     <!-- Body -->
     <!-- NOTE: approximate as a box with "-y" as forward -->
-    <xacro:macro name="body_inertia" params="mass length width height">
+    <xacro:macro name="body_inertial" params="m l w h">
+        <mass value="${m}"/>
         <inertia
-            ixx="${mass*(height*height + length*length)/12.0}" ixy="0.0" ixz="0.0"
-            iyx="0.0" iyy="${mass*(width*width + height*height)/12.0}" iyz="0.0"
-            izx="0.0" izy="0.0" izz="${mass*(width*width + length*length)/12.0}"
+            ixx="${m*(h*h + l*l)/12}" ixy="0" ixz="0"
+            iyy="${m*(w*w + h*h)/12}" iyz="0"
+            izz="${m*(w*w + l*l)/12}"
         />
     </xacro:macro>
     <!-- Wheel -->
     <!-- NOTE: wheels are radially symmetric around the x-axis -->
-    <xacro:macro name="wheel_inertia" params="mass length radius">
+    <xacro:macro name="wheel_inertial" params="m r h">
+        <mass value="${m}"/>
         <inertia
-            ixx="${mass*radius*radius/2.0}" ixy="0.0" ixz="0.0"
-            iyx="0.0" iyy="${mass*(3*radius*radius + length*length)/12.0}" iyz="0.0"
-            izx="0.0" izy="0.0" izz="${mass*(3*radius*radius + length*length)/12.0}"
-        />
-    </xacro:macro>
-    <!-- Sphere -->
-    <xacro:macro name="sphere_inertia" params="mass radius">
-        <inertia
-            ixx="${(2.0 * mass * radius * radius) / 5.0}" ixy="0.0" ixz="0.0"
-            iyx="0.0" iyy="${(2.0 * mass * radius * radius) / 5.0}" iyz="0.0"
-            izx="0.0" izy="0.0" izz="${(2.0 * mass * radius * radius) / 5.0}"
+            ixx="${m*r*r/2}" ixy="0" ixz="0"
+            iyy="${m*(3*r*r + h*h)/12}" iyz="0"
+            izz="${m*(3*r*r + h*h)/12}"
         />
     </xacro:macro>

File: description/urdf/plugins.gazebo.xacro (robot description, xacro)
@@ -3,5 +3,4 @@
     <!-- Constants -->
     <xacro:include filename="$(find description)/urdf/constants.xacro"/>
-    <!-- TODO: ensure we can turn properly! -->
     <!-- Differential Drive Controller -->
     <gazebo>
@@ -9,5 +8,5 @@
             <alwaysOn>true</alwaysOn>
             <legacyMode>false</legacyMode>
-            <rosDebugLevel>na</rosDebugLevel> -->
+            <rosDebugLevel>na</rosDebugLevel>
             <!-- Plugin update rate (Hz) -->
             <updateRate>30</updateRate>
@@ -41,28 +40,31 @@
     </gazebo>
     <!-- IR Sensor: Range Sensor -->
+    <xacro:property name="range_sensor_fov" value="${5*pi/180}"/>
+    <xacro:property name="range_sensor_update_rate" value="50"/>
+    <xacro:property name="range_sensor_max_range" value="0.8"/>
     <gazebo reference="base_ir_link">
         <sensor type="ray" name="RangeSensor">
             <pose>0 0 0 0 0 0</pose>
             <visualize>false</visualize>
-            <update_rate>50</update_rate>
+            <update_rate>${range_sensor_update_rate}</update_rate>
             <ray>
                 <scan>
-                <horizontal>
-                    <samples>10</samples>
-                    <resolution>1</resolution>
-                    <min_angle>-0.14835</min_angle>
-                    <max_angle>0.14835</max_angle>
-                </horizontal>
-                <vertical>
-                    <samples>10</samples>
-                    <resolution>1</resolution>
-                    <min_angle>-0.14835</min_angle>
-                    <max_angle>0.14835</max_angle>
-                </vertical>
+                    <horizontal>
+                        <samples>10</samples>
+                        <resolution>1</resolution>
+                        <min_angle>${-range_sensor_fov/2}</min_angle>
+                        <max_angle>${range_sensor_fov/2}</max_angle>
+                    </horizontal>
+                    <vertical>
+                        <samples>10</samples>
+                        <resolution>1</resolution>
+                        <min_angle>${-range_sensor_fov/2}</min_angle>
+                        <max_angle>${range_sensor_fov/2}</max_angle>
+                    </vertical>
                 </scan>
                 <range>
-                <min>0.01</min>
-                <max>2</max>
-                <resolution>0.02</resolution>
+                    <min>0.01</min>
+                    <max>10</max>
+                    <resolution>0.02</resolution>
                 </range>
             </ray>
@@ -70,14 +72,13 @@
                 <gaussianNoise>0.005</gaussianNoise>
                 <alwaysOn>true</alwaysOn>
-                <updateRate>50</updateRate>
+                <updateRate>${range_sensor_update_rate}</updateRate>
                 <topicName>sensor/ir</topicName>
                 <frameName>base_ir_link</frameName>
                 <radiation>INFRARED</radiation>
-                <fov>0.2967</fov>
+                <fov>${range_sensor_fov}</fov>
             </plugin>
         </sensor>
     </gazebo>
     <!-- Illuminance Sensor: Inherits from Camera -->
-    <!-- NOTE: illuminance only published if the image topic is being read from! -->
     <gazebo reference="light_link">
         <sensor name='light_sensor' type='camera'>
@@ -97,5 +98,5 @@
                 <cameraName>light_sensor</cameraName>
                 <alwaysOn>true</alwaysOn>
-                <updateRate>10</updateRate>
+                <updateRate>50</updateRate>
                 <imageTopicName>rgb/image_raw</imageTopicName>
                 <depthImageTopicName>depth/image_raw</depthImageTopicName>

File: description/urdf/wheels.urdf.xacro (robot description, xacro)
@@ -6,5 +6,5 @@
     <!-- Motor Transmissions -->
     <xacro:macro name="Transmission" params="joint">
-        <transmission name="trans_${joint}">
+        <transmission name="${joint}_trans">
             <type>transmission_interface/SimpleTransmission</type>
             <joint name="${joint}">
@@ -16,4 +16,5 @@
     <!-- Wheel macro -->
     <xacro:macro name="Wheel" params="fb lr">
+        <!-- Wheel link -->
         <link name="${fb}_${lr}_wheel_link">
             <visual>
@@ -26,12 +27,12 @@
                 <origin xyz="0 0 0" rpy="0 ${pi/2} 0"/>
                 <geometry>
-                    <cylinder length="${wheel_width}" radius="${wheel_radius}"/>
+                    <cylinder radius="${wheel_radius}" length="${wheel_width}"/>
                 </geometry>
             </collision>
             <inertial>
-                <mass value="${wheel_mass}"/>
-                <xacro:wheel_inertia mass="${wheel_mass}" length="${wheel_width}" radius="${wheel_radius}"/>
+                <xacro:wheel_inertial m="${wheel_mass}" r="${wheel_radius}" h="${wheel_width}"/>
             </inertial>
         </link>
+        <!-- Wheel joint -->
         <joint name="${fb}_${lr}_wheel_joint" type="continuous">
             <parent link="body_link"/>
@@ -40,10 +41,21 @@
             <axis xyz="1 0 0"/>
         </joint>
-        <xacro:Transmission joint="${fb}_${lr}_wheel_joint"/>
+        <!-- Other attributes-->
+        <xacro:if value="${fb == 'front'}">
+            <!-- Add Transmission to Wheels connected to the motor -->
+            <xacro:Transmission joint="${fb}_${lr}_wheel_joint"/>
+        </xacro:if>
+        <xacro:if value="${fb == 'back'}">
+            <!-- Other Wheels serve for balance only, remove friction to enable turning -->
+            <gazebo reference ="${fb}_${lr}_wheel_link">
+                <mu1 value="0.0"/>
+                <mu2 value="0.0"/>
+            </gazebo>
+        </xacro:if>
     </xacro:macro>
     <!-- Instantiate wheels -->
     <xacro:Wheel fb="front" lr="left"/>
+    <xacro:Wheel fb="front" lr="right"/>
     <xacro:Wheel fb="back" lr="left"/>
-    <xacro:Wheel fb="front" lr="right"/>
     <xacro:Wheel fb="back" lr="right"/>
 </robot>
